File: hardware/irrigation-sensor/irrgiation-sensor-rev4-2.kicad_pcb (KiCad board)
At the start: 2 copper layers, 180 x 38 mm, 39 parts, among them J1 CONUFL001-SMD-T, J2 SHF-105-01-L-D-TH, Q1 TSM260P02, Q2 PMV250EPEA, U1 24LC32, U2 RFM95W, U3 STM32L412KB, U4 TLV61225, Y1 32768Hz

Commit message: Add different irrigation sensor hardware revisions and cypress e2e tests
Routing:
- net SENSOR_PLANE: track 23.3 -> 43.3 mm
Other:
- board text added: "JLCJLCJLCJLC"
- board text added: "Prosper III Pflanzenmonitor rev.4/2"
- board text removed: "Prosper III Pflanzenmonitor rev.4/1"
